Commit message: Se modifico la inercia del base_link en el archivo robotfr.xacro para simularlo en Gazebo. Se cambio de 10 a 1000 en ixx, iyy e izz

File: urdf/robotfr.xacro (robot description, xacro)
@@ -11,5 +11,5 @@
       <origin xyz="0.00072554 2.2065E-05 0.024268" rpy="0 0 0" />
       <mass value="0.01" />
-      <inertia ixx="10" ixy="0" ixz="0" iyy="10" iyz="0" izz="10" />
+      <inertia ixx="1000" ixy="0" ixz="0" iyy="1000" iyz="0" izz="1000" />
     </inertial>
     <!-- Visualizacion del robot-->
